File: HD3SS215.kicad_sch (KiCad schematic)
At the start: 8 parts

Commit message: Adding 5v and 3v3 buck
Parts:
- added C? (x10): 0.1u, symbol Device:C_Small
Connections:
- net DP_C.AUX_M: now also C?.2; no longer U?.14 (AUXA_M)
- net DP_C.AUX_P: now also C?.2; no longer U?.13 (AUXC_P)
- net DP_C.D0_M: now also C?.2; no longer U?.3 (DC0_M)
- net DP_C.D0_P: now also C?.2; no longer U?.2 (DC0_P)
- net DP_C.D1_M: now also C?.2; no longer U?.6 (DC1_M)
- net DP_C.D1_P: now also C?.2; no longer U?.5 (DC1_P)
- net DP_C.D2_M: now also C?.2; no longer U?.9 (DC2_M)
- net DP_C.D2_P: now also C?.2; no longer U?.8 (DC2_P)
- net DP_C.D3_M: now also C?.2; no longer U?.12 (DC3_M)
- net DP_C.D3_P: now also C?.2; no longer U?.11 (DC3_P)
- new net: C?.1, U?.14 (AUXA_M)
- new net: C?.1, U?.3 (DC0_M)
- new net: C?.1, U?.9 (DC2_M)
- new net: C?.1, U?.6 (DC1_M)
- new net: C?.1, U?.12 (DC3_M)
- new net AUXC_P: C?.1, U?.13 (AUXC_P)
- new net DPC_D0_P: C?.1, U?.2 (DC0_P)
- new net DPC_D1_P: C?.1, U?.5 (DC1_P)
- new net DPC_D2_P: C?.1, U?.8 (DC2_P)
- new net DPC_D3_P: C?.1, U?.11 (DC3_P)

Commit message: Fixing ERC
Parts:
- added R12, R13, R14, R15, R17, R18: 4.7k, symbol Device:R_US
- U1: renamed from U?; footprint (none) -> Package_DFN_QFN:QFN-56-1EP_8x8mm_P0.5mm_EP4.5x5.2mm_ThermalVias
- gave numbers to parts that had none: 16
Connections:
- net +3V3: now also R12.1, R13.1, R14.1, R15.1, R17.1, R18.1
- net DP_A.DDCCLK renamed A_DDCCLK
- net A_DDCCLK: now also R14.2
- net DP_A.DDCDAT renamed A_DDCDAT
- net A_DDCDAT: now also R12.2
- net DP_B.DDCCLK renamed B_DDCCLK
- net B_DDCCLK: now also R15.2
- net DP_B.DDCDAT renamed B_DDCDAT
- net B_DDCDAT: now also R13.2
- net DP_C.DDCCLK renamed C_DDCCLK
- net C_DDCCLK: now also R17.2
- net DP_C.DDCDAT renamed C_DDCDAT
- net C_DDCDAT: now also R18.2
