File: InConn.kicad_sch (KiCad schematic)
At the start: 0 parts

Commit message: Adding 5v and 3v3 buck
Parts:
- added J?: 2041441-1, TE_2041441-1, symbol 2041441-1:DP_CONN
- added J?: USB_C_Receptacle_USB2.0, symbol Connector:USB_C_Receptacle_USB2.0
- added R? (x2): 5.1k, symbol Device:R_US
- added R?: 0, symbol Device:R_US
- added R?: 1M, symbol Device:R_US
- added R?: 5M, symbol Device:R_US
Connections:
- new net: J?.B5 (CC2), R?.1
- new net: J?.20 (DP_PWR), R?.2
- new net: J?.13 (CFG1), R?.1
- new net: J?.14 (CFG2), R?.1
- new net: J?.A5 (CC1), R?.1
- new net +3V3: R?.1
- new net GND: J?.11 (GND), J?.16 (GND), J?.19 (RTN), J?.2 (GND), J?.5 (GND), J?.8 (GND), J?.A1 (GND), J?.A12 (GND), J?.B1 (GND), J?.B12 (GND), J?.S1 (SHIELD), J?.SH1 (SHIELD), J?.SH2 (SHIELD), J?.SH3 (SHIELD), R?.2, R?.2, R?.2, R?.2
- new net SOURCE_DP.AUX_M: J?.17 (AUX_N)
- new net SOURCE_DP.AUX_P: J?.15 (AUX_P)
- new net SOURCE_DP.D0_M: J?.3 (ML0_M)
- new net SOURCE_DP.D0_P: J?.1 (ML0_P)
- new net SOURCE_DP.D1_M: J?.6 (ML1_N)
- new net SOURCE_DP.D1_P: J?.4 (ML1_P)
- new net SOURCE_DP.D2_M: J?.9 (ML2_M)
- new net SOURCE_DP.D2_P: J?.7 (ML2_P)
- new net SOURCE_DP.D3_M: J?.12 (ML3_N)
- new net SOURCE_DP.D3_P: J?.10 (ML3_P)
- new net SOURCE_DP.HPD: J?.18 (HPD)
- new net SOURCE_USB.D_M: J?.A7 (D-), J?.B7 (D-)
- new net SOURCE_USB.D_P: J?.A6 (D+), J?.B6 (D+)
- new net VBUS: J?.A4 (VBUS), J?.A9 (VBUS), J?.B4 (VBUS), J?.B9 (VBUS)
- no-connect marks 0 -> 2

Commit message: Fixing ERC
Parts:
- gave numbers to parts that had none: 7
Changed lines of the file:
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@@
   (symbol (lib_id "Device:R_US") (at 167.9194 155.0162 0) (unit 1)
     (in_bom yes) (on_board yes)
-    (property "Reference" "R?" (id 0) (at 163.6776 153.8986 0)
+    (property "Reference" "R4" (id 0) (at 163.6776 153.8986 0)
       (effects (font (size 1.27 1.27)) (justify left))
     )
@@
   (symbol (lib_id "power:GND") (at 131.3942 150.9268 0) (unit 1)
     (in_bom yes) (on_board yes) (fields_autoplaced)
-    (property "Reference" "#PWR?" (id 0) (at 131.3942 157.2768 0)
+    (property "Reference" "#PWR06" (id 0) (at 131.3942 157.2768 0)
       (effects (font (size 1.27 1.27)) hide)
     )
@@
   (symbol (lib_id "power:+3V3") (at 113.919 33.0708 0) (mirror y) (unit 1)
     (in_bom yes) (on_board yes) (fields_autoplaced)
-    (property "Reference" "#PWR?" (id 0) (at 113.919 36.8808 0)
+    (property "Reference" "#PWR04" (id 0) (at 113.919 36.8808 0)
       (effects (font (size 1.27 1.27)) hide)
     )
@@
   (symbol (lib_id "power:GND") (at 168.6052 88.1126 0) (mirror y) (unit 1)
     (in_bom yes) (on_board yes) (fields_autoplaced)
-    (property "Reference" "#PWR?" (id 0) (at 168.6052 94.4626 0)
+    (property "Reference" "#PWR010" (id 0) (at 168.6052 94.4626 0)
       (effects (font (size 1.27 1.27)) hide)
     )
@@
   (symbol (lib_id "Device:R_US") (at 113.919 39.0144 0) (unit 1)
     (in_bom yes) (on_board yes)
-    (property "Reference" "R?" (id 0) (at 110.4138 37.8714 0)
+    (property "Reference" "R2" (id 0) (at 110.4138 37.8714 0)
       (effects (font (size 1.27 1.27)) (justify left))
     )
@@
   (symbol (lib_id "Device:R_US") (at 168.6052 84.3026 0) (mirror y) (unit 1)
     (in_bom yes) (on_board yes) (fields_autoplaced)
-    (property "Reference" "R?" (id 0) (at 166.7002 83.0325 0)
+    (property "Reference" "R5" (id 0) (at 166.7002 83.0325 0)
       (effects (font (size 1.27 1.27)) (justify left))
     )
@@
   (symbol (lib_id "Device:R_US") (at 157.3784 84.455 0) (mirror y) (unit 1)
     (in_bom yes) (on_board yes) (fields_autoplaced)
-    (property "Reference" "R?" (id 0) (at 155.2702 83.1849 0)
+    (property "Reference" "R3" (id 0) (at 155.2702 83.1849 0)
       (effects (font (size 1.27 1.27)) (justify left))
     )
@@
   (symbol (lib_id "power:GND") (at 171.2468 158.9532 0) (unit 1)
     (in_bom yes) (on_board yes)
-    (property "Reference" "#PWR?" (id 0) (at 171.2468 165.3032 0)
+    (property "Reference" "#PWR011" (id 0) (at 171.2468 165.3032 0)
       (effects (font (size 1.27 1.27)) hide)
     )
@@
   (symbol (lib_id "Device:R_US") (at 171.2468 155.1432 0) (mirror y) (unit 1)
     (in_bom yes) (on_board yes)
-    (property "Reference" "R?" (id 0) (at 175.4886 154.0256 0)
+    (property "Reference" "R6" (id 0) (at 175.4886 154.0256 0)
       (effects (font (size 1.27 1.27)) (justify left))
     )
@@
   (symbol (lib_id "power:GND") (at 137.033 83.4898 0) (mirror y) (unit 1)
     (in_bom yes) (on_board yes) (fields_autoplaced)
-    (property "Reference" "#PWR?" (id 0) (at 137.033 89.8398 0)
+    (property "Reference" "#PWR07" (id 0) (at 137.033 89.8398 0)
       (effects (font (size 1.27 1.27)) hide)
     )
@@
   (symbol (lib_id "2041441-1:DP_CONN") (at 126.873 63.9572 0) (mirror y) (unit 1)
     (in_bom yes) (on_board yes)
-    (property "Reference" "J?" (id 0) (at 126.8476 37.592 0))
+    (property "Reference" "J1" (id 0) (at 126.8476 37.592 0))
     (property "Value" "2041441-1" (id 1) (at 126.6444 39.8018 0))
     (property "Footprint" "TE_2041441-1" (id 2) (at 126.873 58.6232 0)
@@
   (symbol (lib_id "power:GND") (at 157.3784 88.265 0) (mirror y) (unit 1)
     (in_bom yes) (on_board yes) (fields_autoplaced)
-    (property "Reference" "#PWR?" (id 0) (at 157.3784 94.615 0)
+    (property "Reference" "#PWR08" (id 0) (at 157.3784 94.615 0)
       (effects (font (size 1.27 1.27)) hide)
     )
@@
   (symbol (lib_id "power:GND") (at 167.9194 158.8262 0) (unit 1)
     (in_bom yes) (on_board yes)
-    (property "Reference" "#PWR?" (id 0) (at 167.9194 165.1762 0)
+    (property "Reference" "#PWR09" (id 0) (at 167.9194 165.1762 0)
       (effects (font (size 1.27 1.27)) hide)
     )
@@
   (symbol (lib_id "power:GND") (at 114.4524 54.8132 0) (mirror y) (unit 1)
     (in_bom yes) (on_board yes) (fields_autoplaced)
-    (property "Reference" "#PWR?" (id 0) (at 114.4524 61.1632 0)
+    (property "Reference" "#PWR05" (id 0) (at 114.4524 61.1632 0)
       (effects (font (size 1.27 1.27)) hide)
     )
@@
   (symbol (lib_id "Connector:USB_C_Receptacle_USB2.0") (at 135.255 128.0668 0) (unit 1)
     (in_bom yes) (on_board yes) (fields_autoplaced)
-    (property "Reference" "J?" (id 0) (at 135.255 105.41 0))
+    (property "Reference" "J2" (id 0) (at 135.255 105.41 0))
     (property "Value" "USB_C_Receptacle_USB2.0" (id 1) (at 135.255 107.95 0))
     (property "Footprint" "" (id 2) (at 139.065 128.0668 0)

Commit message: Pushing what i have now
Parts:
- removed J1: 2041441-1, TE_2041441-1, symbol 2041441-1:DP_CONN
- removed J2: USB_C_Receptacle_USB2.0, symbol Connector:USB_C_Receptacle_USB2.0
- removed R2: 0, symbol Device:R_US
- removed R4: 5.1k, symbol Device:R_US
- removed R5: 1M, symbol Device:R_US
- added D1: ${Color}, Diode_SMD:D_0805_2012Metric_Pad1.15x1.40mm_HandSolder, symbol Rockerrobotics:Diodes/754-2043-1-ND
- added P1: USB_C_Plug_USB2.0, Rockerrobotics:AMPHENOL_12402012E212A, symbol Rockerrobotics:Connectors/664-12402012E212ADKR-ND
- R2: renamed from R6; footprint (none) -> Resistor_SMD:R_0603_1608Metric_Pad0.98x0.95mm_HandSolder
- R3: value 5M -> 120; footprint (none) -> Resistor_SMD:R_0603_1608Metric_Pad0.98x0.95mm_HandSolder
Connections:
- net GND: now also D1.1 (K), P1.A1 (GND), P1.A12 (GND), P1.B1 (GND), P1.B12 (GND), P1.S1 (SHIELD); no longer R3.2
- net SOURCE_USB.D_P: now also P1.A6 (D+)
- net VBUS: now also R3.2, P1.A4 (VBUS), P1.A9 (VBUS), P1.B4 (VBUS), P1.B9 (VBUS)
- net at R3.1: now also D1.2 (A)
- net at R2.1: now also P1.A5 (CC)
- new net SOURCE_USB.D_N: P1.A7 (D-)
- no-connect marks 2 -> 1
Other:
- moved on the sheet: R2
